File: CFL_EE_FeatherDebugShield.kicad_pcb (KiCad board)
At the start: 2 copper layers, 33 x 61 mm, 9 parts, among them J1 Conn_01x12, J2 Conn_01x16, J3 CONN_JUMPER_NO, J4 Conn_ARM_JTAG_SWD_10, J5 SWDIO, J6 SWCLK, J7 CONN_JUMPER_NO, J8 CONN_JUMPER_NO, J9 CONN_JUMPER_NO

Commit message: minor mods sch and pcb. version bump to v01b
Other:
- board text added: "Connected Future Labs"
- board text added: "v01b"
- board text removed: "v01a"
Changed lines of the file:
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@@
   (title_block
     (title "FeatherDebugShield")
-    (date "2023-10-23")
-    (rev "v01a")
+    (date "2023-11-10")
+    (rev "v01b")
     (company "Connected Future Labs")
     (comment 1 "Designed by NN")
@@
   (gr_line (start 83.82 101.6) (end 83.82 59.055)
     (stroke (width 0.1) (type default)) (layer "Edge.Cuts"))
-  (gr_text "v01a" (at 107.95 46.99 90) (layer "F.Cu")
+  (gr_text "Connected Future Labs" (at 96.52 99.06) (layer "F.Cu")
+    (effects (font (size 0.75 0.75) (thickness 0.15) bold) (justify bottom))
+  )
+  (gr_text "v01b" (at 107.95 46.99 90) (layer "F.Cu")
     (effects (font (size 1.5 1.5) (thickness 0.3) bold) (justify left bottom))
   )
-  (gr_text "v01a" (at 107.95 46.99 90) (layer "F.SilkS")
+  (gr_text "v01b" (at 107.95 46.99 90) (layer "F.SilkS")
     (effects (font (size 1.5 1.5) (thickness 0.3) bold) (justify left bottom))
   )
+  (gr_text "Connected Future Labs" (at 96.52 99.06) (layer "F.SilkS")
+    (effects (font (size 0.75 0.75) (thickness 0.15) bold) (justify bottom))
+  )
   (gr_text "3D linkage for the part changed.\nThis may cause a DRC {dblquote}part not same as library warning{dblquote}" (at 91.44 71.628) (layer "Cmts.User")
