File: CFL_EE_FeatherDebugShield.kicad_sch (KiCad schematic)
At the start: 9 parts, among them J1 Conn_01x12, J2 Conn_01x16, J3 CONN_JUMPER_NO, J4 Conn_ARM_JTAG_SWD_10, J5 SWDIO, J6 SWCLK, J7 CONN_JUMPER_NO, J8 CONN_JUMPER_NO, J9 CONN_JUMPER_NO

Commit message: minor mods sch and pcb. version bump to v01b
Other:
- note added: "Calculation for connector height and pogo height: This height was emperically calculated to be ~11.5mm. (the theoretical calculation is not completely accurate since the pin's travel inside the female side is not specified) The pogo's height can lie between 10.795mm(0.425mils) and 12.192mm(0.48mils) (calculated using datasheet) Since the height of the connector lies between the pogo's actuation s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"
- note added: "Pogo connectors to contact the SWD pads located on the Feather M0 bottom layer."
- note added: "We cannot use the debugger on ESP32 (for emotibit) as ESP32 pins cannot be simultaneously used for debugging and as IOs by the program. 1. GPIO13 : I2C clock 2. GPIO12 : EmotiBit button 3. GPIO15 : NC 4. GPIO14 : BMI_INT1"
- note removed: "Pogo connectors to contact the SWD points located on the Feather M0 bottom layer."
- note removed: "This height was emperically calculated to be ~11.5mm. (the theoretical calculation is not completely accurate since the pin's travel inside the female side is not specified) The pogo's height can lie between 10.795mm(0.425mils) and 12.192mm(0.48mils) (calculated using datasheet) Since the height of the connector lies between the pogo's actuation span, a good contact should be made"
- note removed: "We cannot use the debugger on ESP32 as ESP32 pins cannot be simultaneously used for debugging and as IOs by the program. 1. GPIO13 : I2C clock 2. GPIO12 : EmotiBit button 3. GPIO15 : NC 4. GPIO14 : BMI_INT1"
- note removed: "depth unknown"
Changed lines of the file:
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@@
   (title_block
     (title "FeatherDebugShield")
-    (date "2023-10-23")
-    (rev "v01a")
+    (date "2023-11-10")
+    (rev "v01b")
     (company "Connected Future Labs")
     (comment 1 "Designed by NN")
@@
     (stroke (width 0) (type default))
   )
-  (polyline (pts (xy 95.631 66.929) (xy 95.885 66.675))
-    (stroke (width 0) (type default))
-  )
   (wire (pts (xy 91.44 130.81) (xy 107.95 130.81))
     (stroke (width 0) (type default))
@@
     (stroke (width 0) (type default))
   )
-  (polyline (pts (xy 99.06 67.31) (xy 100.33 66.04))
-    (stroke (width 0) (type default))
-  )
   (wire (pts (xy 53.34 96.52) (xy 53.34 100.33))
     (stroke (width 0) (type default))
@@
     (stroke (width 0) (type default))
   )
-  (polyline (pts (xy 95.885 66.675) (xy 96.139 66.929))
-    (stroke (width 0) (type default))
-  )
-  (polyline (pts (xy 95.885 67.818) (xy 96.139 67.564))
-    (stroke (width 0) (type default))
-  )
   (wire (pts (xy 91.44 125.73) (xy 104.14 125.73))
     (stroke (width 0) (type default))
   )
-  (polyline (pts (xy 95.885 66.675) (xy 95.885 67.945))
-    (stroke (width 0) (type dot))
-  )
   (polyline (pts (xy 74.295 62.865) (xy 74.93 63.5))
     (stroke (width 0) (type default))
@@
   )
   (wire (pts (xy 91.44 115.57) (xy 104.14 115.57))
-    (stroke (width 0) (type default))
-  )
-  (polyline (pts (xy 95.631 67.564) (xy 95.885 67.818))
     (stroke (width 0) (type default))
   )
@@
   )
   (wire (pts (xy 60.96 100.33) (xy 68.58 100.33))
-    (stroke (width 0) (type default))
-  )
-  (polyline (pts (xy 96.52 67.31) (xy 99.06 67.31))
     (stroke (width 0) (type default))
   )
@@
     (effects (font (size 1.27 1.27)) (justify left bottom) (href "https://docs.espressif.com/projects/esp-idf/en/latest/esp32/api-guides/jtag-debugging/configure-other-jtag.html"))
   )
-  (text "Pogo connectors to contact the SWD points\nlocated on the Feather M0 bottom layer."
+  (text "Pogo connectors to contact the SWD pads\nlocated on the Feather M0 bottom layer."
     (at 66.04 36.83 0)
     (effects (font (size 1.27 1.27)) (justify left bottom))
   )
-  (text "We cannot use the debugger on ESP32 as\nESP32 pins cannot be simultaneously used for debugging\nand as IOs by the program.\n1. GPIO13 : I2C clock\n2. GPIO12 : EmotiBit button\n3. GPIO15 : NC\n4. GPIO14 : BMI_INT1"
+  (text "We cannot use the debugger on ESP32 (for emotibit) as\nESP32 pins cannot be simultaneously used for debugging\nand as IOs by the program.\n1. GPIO13 : I2C clock\n2. GPIO12 : EmotiBit button\n3. GPIO15 : NC\n4. GPIO14 : BMI_INT1"
     (at 134.62 128.27 0)
     (effects (font (size 1.27 1.27)) (justify left bottom))
@@
     (effects (font (size 1.27 1.27)) (justify left bottom))
   )
-  (text "This height was emperically calculated to be ~11.5mm.\n(the theoretical calculation is not completely accurate\nsince the pin's travel inside the female side is not specified)\n\nThe pogo's height can lie between \n10.795mm(0.425mils) and 12.192mm(0.48mils)\n(calculated using datasheet)\nSince the height of the connector lies between the pogo's\nactuation span, a good contact should be made"
+  (text "Calculation for connector height and pogo height:\n\nThis height was emperically calculated to be ~11.5mm.\n(the theoretical calculation is not completely accurate\nsince the pin's travel inside the female side is not specified)\n\nThe pogo's height can lie between \n10.795mm(0.425mils) and 12.192mm(0.48mils)\n(calculated using datasheet)\nSince the height of the connector lies between the pogo's\nactuation span, a good contact should be made"
     (at 25.4 72.39 0)
     (effects (font (size 1 1)) (justify left bottom))
@@
     (at 111.76 143.51 0)
     (effects (font (size 1.27 1.27)) (justify left bottom))
-  )
-  (text "depth unknown" (at 100.33 66.04 0)
-    (effects (font (size 0.5 0.5)) (justify left bottom))
   )
   (label "GPIO14" (at 93.98 130.81 0) (fields_autoplaced)
@@
     (pin "1")
     (instances
-      (project "CFL_EmotiBit_DebugShield"
+      (project "CFL_EE_FeatherDebugShield"
         (path "/0051c2d3-6afe-4dfe-a36e-434dbeeb15f1"
           (reference "#FLG02") (unit 1)
@@
     (pin "2")
     (instances
-      (project "CFL_EmotiBit_DebugShield"
+      (project "CFL_EE_FeatherDebugShield"
         (path "/0051c2d3-6afe-4dfe-a36e-434dbeeb15f1"
           (reference "J7") (unit 1)
@@
     (pin "9")
     (instances
-      (project "CFL_EmotiBit_DebugShield"
+      (project "CFL_EE_FeatherDebugShield"
         (path "/0051c2d3-6afe-4dfe-a36e-434dbeeb15f1"
           (reference "J2") (unit 1)
@@
     (pin "2")
     (instances
-      (project "CFL_EmotiBit_DebugShield"
+      (project "CFL_EE_FeatherDebugShield"
         (path "/0051c2d3-6afe-4dfe-a36e-434dbeeb15f1"
           (reference "J3") (unit 1)
@@
     (pin "1")
     (instances
-      (project "CFL_EmotiBit_DebugShield"
+      (project "CFL_EE_FeatherDebugShield"
         (path "/0051c2d3-6afe-4dfe-a36e-434dbeeb15f1"
           (reference "J5") (unit 1)
@@
     (pin "2")
     (instances
-      (project "CFL_EmotiBit_DebugShield"
+      (project "CFL_EE_FeatherDebugShield"
         (path "/0051c2d3-6afe-4dfe-a36e-434dbeeb15f1"
           (reference "J8") (unit 1)
@@
     (pin "2")
     (instances
-      (project "CFL_EmotiBit_DebugShield"
+      (project "CFL_EE_FeatherDebugShield"
         (path "/0051c2d3-6afe-4dfe-a36e-434dbeeb15f1"
           (reference "J9") (unit 1)
@@
     (pin "1")
     (instances
-      (project "CFL_EmotiBit_DebugShield"
+      (project "CFL_EE_FeatherDebugShield"
         (path "/0051c2d3-6afe-4dfe-a36e-434dbeeb15f1"
           (reference "#PWR05") (unit 1)
@@
     (pin "9")
     (instances
-      (project "CFL_EmotiBit_DebugShield"
+      (project "CFL_EE_FeatherDebugShield"
         (path "/0051c2d3-6afe-4dfe-a36e-434dbeeb15f1"
           (reference "J4") (unit 1)
@@
     (pin "1")
     (instances
-      (project "CFL_EmotiBit_DebugShield"
+      (project "CFL_EE_FeatherDebugShield"
         (path "/0051c2d3-6afe-4dfe-a36e-434dbeeb15f1"
           (reference "#FLG01") (unit 1)
@@
     (pin "1")
     (instances
-      (project "CFL_EmotiBit_DebugShield"
+      (project "CFL_EE_FeatherDebugShield"
         (path "/0051c2d3-6afe-4dfe-a36e-434dbeeb15f1"
           (reference "#PWR02") (unit 1)
@@
     (pin "1")
     (instances
-      (project "CFL_EmotiBit_DebugShield"
+      (project "CFL_EE_FeatherDebugShield"
         (path "/0051c2d3-6afe-4dfe-a36e-434dbeeb15f1"
           (reference "#PWR01") (unit 1)
@@
     (pin "9")
     (instances
-      (project "CFL_EmotiBit_DebugShield"
+      (project "CFL_EE_FeatherDebugShield"
         (path "/0051c2d3-6afe-4dfe-a36e-434dbeeb15f1"
           (reference "J1") (unit 1)
@@
     (pin "1")
     (instances
-      (project "CFL_EmotiBit_DebugShield"
+      (project "CFL_EE_FeatherDebugShield"
         (path "/0051c2d3-6afe-4dfe-a36e-434dbeeb15f1"
           (reference "J6") (unit 1)
@@
     (pin "1")
     (instances
-      (project "CFL_EmotiBit_DebugShield"
+      (project "CFL_EE_FeatherDebugShield"
         (path "/0051c2d3-6afe-4dfe-a36e-434dbeeb15f1"
           (reference "#PWR03") (unit 1)
